Commit message: add v-hacd decomposed meshes for collisions

File: ycb_objects_models_sim/objects/YcbBanana/model.urdf (robot description, URDF)
Before this commit: robot model.urdf, 1 links, 0 joints
Links:
- link baseLink: geometry collision mesh filename=collision_vhacd.obj scale=1 1 1; visual mesh filename=textured_simple_reoriented.obj scale=1 1 1

File: ycb_objects_models_sim/objects/YcbChipsCan/model.urdf (robot description, URDF)
Before this commit: robot model.urdf, 1 links, 0 joints
Links:
- link baseLink: geometry collision mesh filename=collision_vhacd.obj scale=1 1 1; visual mesh filename=textured.obj scale=1 1 1

File: ycb_objects_models_sim/objects/YcbCrackerBox/model.urdf (robot description, URDF)
Before this commit: robot model.urdf, 1 links, 0 joints
Links:
- link baseLink: geometry collision mesh filename=collision_vhacd.obj scale=1 1 1; visual mesh filename=textured_simple_reoriented.obj scale=1 1 1

File: ycb_objects_models_sim/objects/YcbFoamBrick/model.urdf (robot description, URDF)
Before this commit: robot model.urdf, 1 links, 0 joints
Links:
- link baseLink: geometry collision mesh filename=collision_vhacd.obj scale=1 1 1; visual mesh filename=textured_simple_reoriented.obj scale=1 1 1

File: ycb_objects_models_sim/objects/YcbGelatinBox/model.urdf (robot description, URDF)
Before this commit: robot model.urdf, 1 links, 0 joints
Links:
- link baseLink: geometry collision mesh filename=collision_vhacd.obj scale=1 1 1; visual mesh filename=textured_simple_reoriented.obj scale=1 1 1

File: ycb_objects_models_sim/objects/YcbHammer/model.urdf (robot description, URDF)
Before this commit: robot model.urdf, 1 links, 0 joints
Links:
- link baseLink: geometry collision mesh filename=collision_vhacd.obj scale=1 1 1; visual mesh filename=textured_simple_reoriented.obj scale=1 1 1

File: ycb_objects_models_sim/objects/YcbMasterChefCan/model.urdf (robot description, URDF)
Before this commit: robot model.urdf, 1 links, 0 joints
Links:
- link baseLink: geometry collision mesh filename=collision_vhacd.obj scale=1 1 1; visual mesh filename=textured_simple_reoriented.obj scale=1 1 1

File: ycb_objects_models_sim/objects/YcbMediumClamp/model.urdf (robot description, URDF)
Before this commit: robot model.urdf, 1 links, 0 joints
Links:
- link baseLink: geometry collision mesh filename=collision_vhacd.obj scale=1 1 1; visual mesh filename=textured_reoriented.obj scale=1 1 1

File: ycb_objects_models_sim/objects/YcbMustardBottle/model.urdf (robot description, URDF)
Before this commit: robot model.urdf, 1 links, 0 joints
Links:
- link baseLink: geometry collision mesh filename=collision_vhacd.obj scale=1 1 1; visual mesh filename=textured_simple_reoriented.obj scale=1 1 1

File: ycb_objects_models_sim/objects/YcbPear/model.urdf (robot description, URDF)
Before this commit: robot model.urdf, 1 links, 0 joints
Links:
- link baseLink: geometry collision mesh filename=collision_vhacd.obj scale=1 1 1; visual mesh filename=textured_simple_reoriented.obj scale=1 1 1

File: ycb_objects_models_sim/objects/YcbPottedMeatCan/model.urdf (robot description, URDF)
Before this commit: robot model.urdf, 1 links, 0 joints
Links:
- link baseLink: geometry collision mesh filename=collision_vhacd.obj scale=1 1 1; visual mesh filename=textured_simple_reoriented.obj scale=1 1 1

File: ycb_objects_models_sim/objects/YcbPowerDrill/model.urdf (robot description, URDF)
Before this commit: robot model.urdf, 1 links, 0 joints
Links:
- link baseLink: geometry collision mesh filename=collision_vhacd.obj scale=1 1 1; visual mesh filename=textured_simple_reoriented.obj scale=1 1 1

File: ycb_objects_models_sim/objects/YcbScissors/model.urdf (robot description, URDF)
Before this commit: robot model.urdf, 1 links, 0 joints
Links:
- link baseLink: geometry collision mesh filename=collision_vhacd.obj scale=1 1 1; visual mesh filename=textured_simple_reoriented.obj scale=1 1 1

File: ycb_objects_models_sim/objects/YcbStrawberry/model.urdf (robot description, URDF)
Before this commit: robot model.urdf, 1 links, 0 joints
Links:
- link baseLink: geometry collision mesh filename=collision_vhacd.obj scale=1 1 1; visual mesh filename=textured_reoriented.obj scale=1 1 1

File: ycb_objects_models_sim/objects/YcbTennisBall/model.urdf (robot description, URDF)
Before this commit: robot model.urdf, 1 links, 0 joints
Links:
- link baseLink: geometry collision mesh filename=collision_vhacd.obj scale=1 1 1; visual mesh filename=textured_reoriented.obj scale=1 1 1

File: ycb_objects_models_sim/objects/YcbTomatoSoupCan/model.urdf (robot description, URDF)
Before this commit: robot model.urdf, 1 links, 0 joints
Links:
- link baseLink: geometry collision mesh filename=collision_vhacd.obj scale=1 1 1; visual mesh filename=textured_simple_reoriented.obj scale=1 1 1
