Commit message: fix weird mesh and reduce vertexes for all objects

File: ycb_objects_models_sim/objects/YcbPear/model.urdf (robot description, URDF)
Before this commit: robot model.urdf, 1 links, 0 joints
Links:
- link baseLink: geometry collision mesh filename=collision_vhacd.obj scale=1 1 1; visual mesh filename=textured_reoriented.obj scale=1 1 1
