Commit message: add custom cylinders for cross-validation experiments

File: ycb_objects_models_sim/objects/MyCylinder_1/model.urdf (robot description, URDF)
Before this commit: robot model.urdf, 1 links, 0 joints
Links:
- link baseLink: mass .082 -> .100; geometry collision mesh filename=mesh.obj scale=1 1 1; visual mesh filename=mesh.obj scale=1 1 1

File: ycb_objects_models_sim/objects/MyCylinder_2/model.urdf (robot description, URDF)
Before this commit: robot model.urdf, 1 links, 0 joints
Links:
- link baseLink: mass .082 -> .100; geometry collision mesh filename=mesh.obj scale=1 1 1; visual mesh filename=mesh.obj scale=1 1 1

File: ycb_objects_models_sim/objects/MyCylinder_3/model.urdf (robot description, URDF)
Before this commit: robot model.urdf, 1 links, 0 joints
Links:
- link baseLink: mass .082 -> .100; geometry collision mesh filename=mesh.obj scale=1 1 1; visual mesh filename=mesh.obj scale=1 1 1

File: ycb_objects_models_sim/objects/MyCylinder_cone_bend_3/model.urdf (robot description, URDF)
Before this commit: robot model.urdf, 1 links, 0 joints
Links:
- link baseLink: mass .082 -> .100; geometry collision mesh filename=mesh.obj scale=1 1 1; visual mesh filename=mesh.obj scale=1 1 1

File: ycb_objects_models_sim/objects/MyCylinder_oval_3/model.urdf (robot description, URDF)
Before this commit: robot model.urdf, 1 links, 0 joints
Links:
- link baseLink: mass .082 -> .100; geometry collision mesh filename=mesh.obj scale=1 1 1; visual mesh filename=mesh.obj scale=1 1 1
