Commit message: improve collision, COM pos and friction for all objects

File: ycb_objects_models_sim/objects/YcbChipsCan/model.urdf (robot description, URDF)
Before this commit: robot model.urdf, 1 links, 0 joints
Links:
- link baseLink: geometry collision mesh filename=collision_vhacd.obj scale=0.95 0.95 1.0; visual mesh filename=textured.obj scale=0.95 0.95 1.0

File: ycb_objects_models_sim/objects/YcbHammer/model.urdf (robot description, URDF)
Before this commit: robot model.urdf, 1 links, 0 joints
Links:
- link baseLink: geometry collision mesh filename=collision_vhacd.obj scale=1 1 1; visual mesh filename=textured_reoriented.obj scale=1 1 1

File: ycb_objects_models_sim/objects/YcbMasterChefCan/model.urdf (robot description, URDF)
Before this commit: robot model.urdf, 1 links, 0 joints
Links:
- link baseLink: geometry collision mesh filename=collision_vhacd.obj scale=0.7 0.7 0.7; visual mesh filename=textured_simple_reoriented.obj scale=0.7 0.7 0.7
